Commit message: urdf v4... check

File: EASY/Easy Task3/urdf4/urdf4/urdf/urdf4.urdf (robot description, URDF)
Before this commit: robot Assem1, 5 links, 4 joints
Links:
- link LF: mass 0.0489436503728706 -> 0.048944; geometry collision mesh filename=package://urdf4/meshes/LF.STL; visual mesh filename=package://urdf4/meshes/LF.STL
- link LR: mass 0.0489436503728706 -> 0.048944; geometry collision mesh filename=package://urdf4/meshes/LR.STL; visual mesh filename=package://urdf4/meshes/LR.STL
- link RB: mass 0.0489436503728706 -> 0.048944; geometry collision mesh filename=package://urdf4/meshes/RB.STL; visual mesh filename=package://urdf4/meshes/RB.STL
- link RF: mass 0.0489436503728706 -> 0.048944; geometry collision mesh filename=package://urdf4/meshes/RF.STL; visual mesh filename=package://urdf4/meshes/RF.STL
- link base_link: mass 0.734157679226464 -> 0.73416; geometry collision mesh filename=package://urdf4/meshes/base_link.STL; visual mesh filename=package://urdf4/meshes/base_link.STL
Joints:
- joint LRJ: origin xyz=-0.075 -0.06 0.01 rpy=1.5707963267949 -0.584056750958047 1.5707963267949 -> xyz=-0.075 -0.06 0.01 rpy=1.5708 -0.58406 1.5708

File: EASY/Easy Task3/urdf5/urdf5/urdf/urdf5.urdf (robot description, URDF)
Before this commit: robot Assem1, 5 links, 4 joints
Links:
- link LF: geometry collision mesh filename=package://urdf5/meshes/LF.STL; visual mesh filename=package://urdf5/meshes/LF.STL
- link LR: geometry collision mesh filename=package://urdf5/meshes/LR.STL; visual mesh filename=package://urdf5/meshes/LR.STL
- link RB: geometry collision mesh filename=package://urdf5/meshes/RB.STL; visual mesh filename=package://urdf5/meshes/RB.STL
- link RF: geometry collision mesh filename=package://urdf5/meshes/RF.STL; visual mesh filename=package://urdf5/meshes/RF.STL
- link base_link: mass 0.734157679226464 -> 0.734157679226463; geometry collision mesh filename=package://urdf5/meshes/base_link.STL; visual mesh filename=package://urdf5/meshes/base_link.STL
Joints:
- joint LFJ: origin xyz=-0.075 0.05 0.01 rpy=1.5708 0.91772 1.5708 -> xyz=-0.075 0.05 0.01 rpy=1.5707963267949 0.917718602617513 1.5707963267949
- joint RBJ: origin xyz=0.075 -0.06 0.01 rpy=-1.5708 0 -1.5708 -> xyz=0.075 -0.06 0.01 rpy=-1.5707963267949 0 -1.5707963267949
- joint RFJ: origin xyz=0.075 0.05 0.01 rpy=-1.5708 0 -1.5708 -> xyz=0.075 0.05 0.01 rpy=-1.5707963267949 0 -1.5707963267949

File: EASY/Easy Task3/urdf6/urdf6/urdf/urdf6.urdf (robot description, URDF)
Before this commit: robot Assem1, 5 links, 4 joints
Links:
- link LF: geometry collision mesh filename=package://urdf6/meshes/LF.STL; visual mesh filename=package://urdf6/meshes/LF.STL
- link LR: mass 0.0489436503728706 -> 0; geometry collision mesh filename=package://urdf6/meshes/LR.STL; visual mesh filename=package://urdf6/meshes/LR.STL
- link RB: geometry collision mesh filename=package://urdf6/meshes/RB.STL; visual mesh filename=package://urdf6/meshes/RB.STL
- link RF: geometry collision mesh filename=package://urdf6/meshes/RF.STL; visual mesh filename=package://urdf6/meshes/RF.STL
- link base_link: mass 0.734157679226464 -> 0.73416; geometry collision mesh filename=package://urdf6/meshes/base_link.STL; visual mesh filename=package://urdf6/meshes/base_link.STL

File: EASY/Easy Task3/urdf7/urdf7/urdf/urdf7.urdf (robot description, URDF)
Before this commit: robot Assem1, 5 links, 4 joints
Links:
- link LF: geometry collision mesh filename=package://urdf7/meshes/LF.STL; visual mesh filename=package://urdf7/meshes/LF.STL
- link LR: geometry collision mesh filename=package://urdf7/meshes/LR.STL; visual mesh filename=package://urdf7/meshes/LR.STL
- link RB: geometry collision mesh filename=package://urdf7/meshes/RB.STL; visual mesh filename=package://urdf7/meshes/RB.STL
- link RF: geometry collision mesh filename=package://urdf7/meshes/RF.STL; visual mesh filename=package://urdf7/meshes/RF.STL
- link base_link: mass 0.734157679226464 -> 0.73416; geometry collision mesh filename=package://urdf7/meshes/base_link.STL; visual mesh filename=package://urdf7/meshes/base_link.STL
Joints:
- joint LFJ: origin xyz=-0.075 0.05 0.01 rpy=1.5708 0.91772 1.5708 -> xyz=-0.075 0.05 0.01 rpy=1.5707963267949 0.917718602617513 1.5707963267949
- joint RBJ: origin xyz=0.075 -0.06 0.01 rpy=-1.5708 0 -1.5708 -> xyz=0.075 -0.06 0.01 rpy=-1.5707963267949 0 -1.5707963267949
- joint RFJ: origin xyz=0.075 0.05 0.01 rpy=-1.5708 0 -1.5708 -> xyz=0.075 0.05 0.01 rpy=-1.5707963267949 0 -1.5707963267949
