Commit message: floor design3

File: EASY/Easy Task3/project2/protos/floorassemblr12345578.urdf (robot description, URDF)
Before this commit: robot floorassemblr _1009, 2 links, 1 joints
Links:
- link base_link: geometry collision mesh filename=package://floorassemblr12345578/meshes/base_link.STL; visual mesh filename=package://floorassemblr12345578/meshes/base_link.STL
- link fsdf: geometry collision mesh filename=package://floorassemblr12345578/meshes/fsdf.STL; visual mesh filename=package://floorassemblr12345578/meshes/fsdf.STL
