Commit message: floor design4567

File: EASY/Easy Task3/floorassemblr1048/urdf/floorassemblr1048.urdf (robot description, URDF)
Before this commit: robot floorassemblr12345578, 2 links, 1 joints
Links:
- removed link fsdf
- added link dfsdf, mass 5; collision mesh filename=package://floorassemblr1048/meshes/dfsdf.STL; visual mesh filename=package://floorassemblr1048/meshes/dfsdf.STL
- link base_link: geometry collision mesh filename=package://floorassemblr1048/meshes/base_link.STL; visual mesh filename=package://floorassemblr1048/meshes/base_link.STL
Joints:
- removed joint sdfsdf
- added joint ser: type planar, parent base_link, child dfsdf, origin xyz=0.64859 -1.6661 0.92708 rpy=1.5708 0 0, axis 0 0 0
